Commit message: feat: parameterize position based joint velocity limits

File: test/fr3.urdf (robot description, URDF)
Before this commit: robot fp3, 10 links, 9 joints
Joints:
- joint fp3_joint1: limit lower=-2.7437 upper=2.7437 effort=87.0 velocity=2.62 -> lower=-2.750100 upper=2.75010 effort=87.0 velocity=2.62
- joint fp3_joint2: limit lower=-1.7837 upper=1.7837 effort=87.0 velocity=2.62 -> lower=-1.791800 upper=1.79180 effort=87.0 velocity=2.62
- joint fp3_joint3: limit lower=-2.9007 upper=2.9007 effort=87.0 velocity=2.62 -> lower=-2.906500 upper=2.90650 effort=87.0 velocity=2.62
- joint fp3_joint4: limit lower=-3.0421 upper=-0.1518 effort=87.0 velocity=2.62 -> lower=-3.048100 upper=-0.1458 effort=87.0 velocity=2.62
- joint fp3_joint5: limit lower=-2.8065 upper=2.8065 effort=12.0 velocity=5.26 -> lower=-2.810100 upper=2.81010 effort=12.0 velocity=5.26
- joint fp3_joint6: limit lower=0.5445 upper=4.5169 effort=12.0 velocity=4.18 -> lower=0.54092 upper=4.52050 effort=12.0 velocity=4.18
- joint fp3_joint7: limit lower=-3.0159 upper=3.0159 effort=12.0 velocity=5.26 -> lower=-3.019600 upper=3.01960 effort=12.0 velocity=5.26

Commit message: hotfix/fixes zero Jacobian calculation for robot model
github issue -> https://github.com/frankarobotics/libfranka/issues/213

chore: hardcode the last link to link8

File: test/fr3.urdf (robot description, URDF)
Before this commit: robot fp3, 10 links, 9 joints
Links:
- removed link fp3_link0
- removed link fp3_link1
- removed link fp3_link2
- removed link fp3_link3
- removed link fp3_link4
- removed link fp3_link5
- removed link fp3_link6
- removed link fp3_link7
- removed link fp3_link8
- added link link0, mass 2.3966; collision mesh filename=package://franka_description/meshes/robot_arms/fr3/collisio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; visual mesh filename=package://franka_description/meshes/robot_arms/fr3/visual/l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
- added link link0_accelerometer_bottom
- added link link0_accelerometer_top
- added link link1, mass 2.9274653454; collision mesh filename=package://franka_description/meshes/robot_arms/fr3/collisio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; visual mesh filename=package://franka_description/meshes/robot_arms/fr3/visual/l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
- added link link1_accelerometer_bottom
- added link link1_accelerometer_top
- added link link2, mass 2.9355370338; collision mesh filename=package://franka_description/meshes/robot_arms/fr3/collisio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; visual mesh filename=package://franka_description/meshes/robot_arms/fr3/visual/l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
- added link link2_accelerometer_bottom
- added link link2_accelerometer_top
- added link link3, mass 2.2449013699; collision mesh filename=package://franka_description/meshes/robot_arms/fr3/collisio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; visual mesh filename=package://franka_description/meshes/robot_arms/fr3/visual/l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
- added link link3_accelerometer_bottom
- added link link3_accelerometer_top
- added link link4, mass 2.6155955791; collision mesh filename=package://franka_description/meshes/robot_arms/fr3/collisio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; visual mesh filename=package://franka_description/meshes/robot_arms/fr3/visual/l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
- added link link4_accelerometer_bottom
- added link link4_accelerometer_top
- added link link5, mass 2.3271207594; collision mesh filename=package://franka_description/meshes/robot_arms/fr3/collisio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; visual mesh filename=package://franka_description/meshes/robot_arms/fr3/visual/l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
- added link link5_accelerometer_bottom
- added link link5_accelerometer_top
- added link link6, mass 1.8170376524; collision mesh filename=package://franka_description/meshes/robot_arms/fr3/collisio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; visual mesh filename=package://franka_description/meshes/robot_arms/fr3/visual/l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
- added link link7, mass 0.6271432862; collision mesh filename=package://franka_description/meshes/robot_arms/fr3/collisio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; visual mesh filename=package://franka_description/meshes/robot_arms/fr3/visual/l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
- added link link8
Joints:
- removed joint base
- removed joint fp3_joint1
- removed joint fp3_joint2
- removed joint fp3_joint3
- removed joint fp3_joint4
- removed joint fp3_joint5
- removed joint fp3_joint6
- removed joint fp3_joint7
- removed joint fp3_joint8
- added joint base_joint: type fixed, parent base, child link0, origin xyz=0 0 0 rpy=0 0 0
- added joint joint1: type revolute, parent link0, child link1, origin xyz=0 0 0.333 rpy=0 0 0, axis 0 0 1, limit lower=-2.750100 upper=2.75010 effort=87.0 velocity=2.62
- added joint joint2: type revolute, parent link1, child link2, origin xyz=0 0 0 rpy=-1.570796326794897 0 0, axis 0 0 1, limit lower=-1.791800 upper=1.79180 effort=87.0 velocity=2.62
- added joint joint3: type revolute, parent link2, child link3, origin xyz=0 -0.316 0 rpy=1.570796326794897 0 0, axis 0 0 1, limit lower=-2.906500 upper=2.90650 effort=87.0 velocity=2.62
- added joint joint4: type revolute, parent link3, child link4, origin xyz=0.0825 0 0 rpy=1.570796326794897 0 0, axis 0 0 1, limit lower=-3.048100 upper=-0.1458 effort=87.0 velocity=2.62
- added joint joint5: type revolute, parent link4, child link5, origin xyz=-0.0825 0.384 0 rpy=-1.570796326794897 0 0, axis 0 0 1, limit lower=-2.810100 upper=2.81010 effort=12.0 velocity=5.26
- added joint joint6: type revolute, parent link5, child link6, origin xyz=0 0 0 rpy=1.570796326794897 0 0, axis 0 0 1, limit lower=0.54092 upper=4.52050 effort=12.0 velocity=4.18
- added joint joint7: type revolute, parent link6, child link7, origin xyz=0.088 0 0 rpy=1.570796326794897 0 0, axis 0 0 1, limit lower=-3.019600 upper=3.01960 effort=12.0 velocity=5.26
- added joint joint8: type fixed, parent link7, child link8, origin xyz=0 0 0.107 rpy=0 0 0
- added joint link0_accelerometer_bottom_joint: type fixed, parent link0, child link0_accelerometer_bottom, origin xyz=0 0 0.06 rpy=0 0 0
- added joint link0_accelerometer_top_joint: type fixed, parent link0, child link0_accelerometer_top, origin xyz=0 0 0.05 rpy=3.14159 0 0
- added joint link1_accelerometer_bottom_joint: type fixed, parent link1, child link1_accelerometer_bottom, origin xyz=0 -0.09 0.0 rpy=-1.5708 0 0
- added joint link1_accelerometer_top_joint: type fixed, parent link1, child link1_accelerometer_top, origin xyz=0 -0.1 0.0 rpy=1.5708 0 0
- added joint link2_accelerometer_bottom_joint: type fixed, parent link2, child link2_accelerometer_bottom, origin xyz=0 -0.14 0 rpy=1.5708 0 0
- added joint link2_accelerometer_top_joint: type fixed, parent link2, child link2_accelerometer_top, origin xyz=0 -0.13 0 rpy=-1.5708 0 0
- added joint link3_accelerometer_bottom_joint: type fixed, parent link3, child link3_accelerometer_bottom, origin xyz=0.0825 0.04 0 rpy=1.5708 0 0
- added joint link3_accelerometer_top_joint: type fixed, parent link3, child link3_accelerometer_top, origin xyz=0.0825 0.05 0 rpy=-1.5708 0 0
- added joint link4_accelerometer_bottom_joint: type fixed, parent link4, child link4_accelerometer_bottom, origin xyz=-0.0825 0.06 0 rpy=-1.5708 0 0
- added joint link4_accelerometer_top_joint: type fixed, parent link4, child link4_accelerometer_top, origin xyz=-0.0825 0.05 0 rpy=1.5708 0 0
- added joint link5_accelerometer_bottom_joint: type fixed, parent link5, child link5_accelerometer_bottom, origin xyz=0 0.1 0 rpy=1.5708 0 0
- added joint link5_accelerometer_top_joint: type fixed, parent link5, child link5_accelerometer_top, origin xyz=0 0.11 0 rpy=-1.5708 0 0
